Commit message: astar finish

File: src/rikibot_gazebo/urdf/gazebo/robot_base.urdf.xacro (robot description, xacro)
@@ -1,39 +1,57 @@
 <?xml version="1.0"?>
 <robot name="robot_base" xmlns:xacro="http://www.ros.org/wiki/xacro">
-    <xacro:property name="PI" value="3.1415926"/>
+    <xacro:property name="PI" value="3.1415926" />
     <xacro:property name="base_link_width" value="0.16" />
     <xacro:property name="base_link_length" value="0.25" />
     <xacro:property name="base_link_height" value="0.05" />
     <xacro:property name="base_link_m" value="0.5" />
-     <xacro:property name="earth_space" value="0.025" />     <xacro:property name="wheel_offset" value="0.08" />
+    <xacro:property name="earth_space" value="0.025" />
+    <xacro:property name="wheel_offset" value="0.08" />
+    <xacro:macro name="Box_inertial_matrix" params="m l w h">
+        <inertial>
+                <mass value="${m}" />
+                <inertia ixx="${m*(h*h + l*l)/12}" ixy = "0" ixz = "0"
+                    iyy="${m*(w*w + l*l)/12}" iyz= "0"
+                    izz="${m*(w*w + h*h)/12}" />
+        </inertial>
+    </xacro:macro>
+    <xacro:macro name="cylinder_inertial_matrix" params="m r h">
+        <inertial>
+            <mass value="${m}" />
+            <inertia ixx="${m*(3*r*r+h*h)/12}" ixy = "0" ixz = "0"
+                iyy="${m*(3*r*r+h*h)/12}" iyz = "0"
+                izz="${m*r*r/2}" />
+        </inertial>
+    </xacro:macro>
     <link name="base_footprint">
-      <visual>
-        <geometry>
-           <box size="0.001 0.001 0.001" />
-        </geometry>
-      </visual>
+        <visual>
+            <geometry>
+                <box size="0.001 0.001 0.001" />
+            </geometry>
+        </visual>
     </link>
     <link name="base_link">
-      <visual>
-        <geometry>
-          <box size="${base_link_width} ${base_link_length} ${base_link_height}"/>
-        </geometry>
-        <origin rpy="0 0 1.57075" xyz="0 0 0"/>
-        <material name="blue">
-          <color rgba="0 .5 .8 1"/>
-        </material>
-      </visual>
-      <collision>
-        <geometry>
-          <box size="${base_link_width} ${base_link_length} ${base_link_height}"/>
-        </geometry>
-        <origin xyz="0 0 0" rpy="0 0 0" />
-      </collision>
-      <xacro:Box_inertial_matrix m="${base_link_m}" w="${base_link_width}" l="${base_link_length}"  h="${base_link_height}" />
+        <visual>
+            <geometry>
+                <box size="${base_link_width} ${base_link_length} ${base_link_height}" />
+            </geometry>
+            <origin rpy="0 0 1.57075" xyz="0 0 0" />
+            <material name="blue">
+                <color rgba="0 .5 .8 1" />
+            </material>
+        </visual>
+        <collision>
+            <geometry>
+                <box size="${base_link_width} ${base_link_length} ${base_link_height}" />
+            </geometry>
+            <origin xyz="0 0 0" rpy="0 0 0" />
+        </collision>
+        <xacro:Box_inertial_matrix m="${base_link_m}" w="${base_link_width}" l="${base_link_length}"
+            h="${base_link_height}" />
     </link>
     <joint name="base_link2base_footprint" type="fixed">
-      <parent link="base_footprint" />
-      <child link="base_link" />
-      <origin xyz="0 0 ${earth_space + base_link_height}" />
+        <parent link="base_footprint" />
+        <child link="base_link" />
+        <origin xyz="0 0 ${earth_space + base_link_height}" />
     </joint>
     <gazebo reference="base_link">
@@ -44,60 +62,62 @@
     <xacro:property name="wheel_m" value="0.05" />
     <xacro:macro name="add_front_wheels" params="name flag">
-    <link name="${name}_wheel">
-        <visual>
-          <geometry>
-            <cylinder radius="${wheel_radius}" length="${wheel_length}" />
-          </geometry>
-          <origin xyz="0.0 0.0 0.0" rpy="${PI / 2} 0.0 0.0" />
-          <material name="black">
-            <color rgba="0 0 0 1"/>
-        </material>
-        </visual>
-        <collision>
-          <geometry>
-            <cylinder radius="${wheel_radius}" length="${wheel_length}" />
-          </geometry>
-          <origin xyz="0.0 0.0 0.0" rpy="${PI / 2} 0.0 0.0" />
-        </collision>
-        <xacro:cylinder_inertial_matrix m="${wheel_m}" r="${wheel_radius}" h="${wheel_length}" />
-    </link>
-    <joint name="${name}_wheel2base_link" type="continuous">
-        <parent link="base_link" />
-        <child link="${name}_wheel" />
-        <origin xyz="${wheel_offset} ${flag * base_link_width/2} ${-(earth_space + base_link_height / 2 - wheel_radius) }" />
-        <axis xyz="0 1 0" />
-    </joint>
-    <gazebo reference="${name}_wheel">
-      <material>Gazebo/Red</material>
-    </gazebo>
+        <link name="${name}_wheel">
+            <visual>
+                <geometry>
+                    <cylinder radius="${wheel_radius}" length="${wheel_length}" />
+                </geometry>
+                <origin xyz="0.0 0.0 0.0" rpy="${PI / 2} 0.0 0.0" />
+                <material name="black">
+                    <color rgba="0 0 0 1" />
+                </material>
+            </visual>
+            <collision>
+                <geometry>
+                    <cylinder radius="${wheel_radius}" length="${wheel_length}" />
+                </geometry>
+                <origin xyz="0.0 0.0 0.0" rpy="${PI / 2} 0.0 0.0" />
+            </collision>
+            <xacro:cylinder_inertial_matrix m="${wheel_m}" r="${wheel_radius}" h="${wheel_length}" />
+        </link>
+        <joint name="${name}_wheel2base_link" type="continuous">
+            <parent link="base_link" />
+            <child link="${name}_wheel" />
+            <origin
+                xyz="${wheel_offset} ${flag * base_link_width/2} ${-(earth_space + base_link_height / 2 - wheel_radius) }" />
+            <axis xyz="0 1 0" />
+        </joint>
+        <gazebo reference="${name}_wheel">
+            <material>Gazebo/Red</material>
+        </gazebo>
     </xacro:macro>
     <xacro:add_front_wheels name="left_front" flag="1" />
     <xacro:add_front_wheels name="right_front" flag="-1" />
     <xacro:macro name="add_back_wheels" params="name flag">
-    <link name="${name}_wheel">
-        <visual>
-          <geometry>
-            <cylinder radius="${wheel_radius}" length="${wheel_length}" />
-          </geometry>
-          <origin xyz="0.0 0.0 0.0" rpy="${PI / 2} 0.0 0.0" />
-          <material name="black" />
-        </visual>
-        <collision>
-          <geometry>
-            <cylinder radius="${wheel_radius}" length="${wheel_length}" />
-          </geometry>
-          <origin xyz="0.0 0.0 0.0" rpy="${PI / 2} 0.0 0.0" />
-        </collision>
-        <xacro:cylinder_inertial_matrix m="${wheel_m}" r="${wheel_radius}" h="${wheel_length}" />
-    </link>
-    <joint name="${name}_wheel2base_link" type="continuous">
-        <parent link="base_link" />
-        <child link="${name}_wheel" />
-        <origin xyz="${-wheel_offset} ${flag * base_link_width/2} ${-(earth_space + base_link_height / 2 - wheel_radius) }" />
-        <axis xyz="0 1 0" />
-    </joint>
-    <gazebo reference="${name}_wheel">
-      <material>Gazebo/Red</material>
-    </gazebo>
+        <link name="${name}_wheel">
+            <visual>
+                <geometry>
+                    <cylinder radius="${wheel_radius}" length="${wheel_length}" />
+                </geometry>
+                <origin xyz="0.0 0.0 0.0" rpy="${PI / 2} 0.0 0.0" />
+                <material name="black" />
+            </visual>
+            <collision>
+                <geometry>
+                    <cylinder radius="${wheel_radius}" length="${wheel_length}" />
+                </geometry>
+                <origin xyz="0.0 0.0 0.0" rpy="${PI / 2} 0.0 0.0" />
+            </collision>
+            <xacro:cylinder_inertial_matrix m="${wheel_m}" r="${wheel_radius}" h="${wheel_length}" />
+        </link>
+        <joint name="${name}_wheel2base_link" type="continuous">
+            <parent link="base_link" />
+            <child link="${name}_wheel" />
+            <origin
+                xyz="${-wheel_offset} ${flag * base_link_width/2} ${-(earth_space + base_link_height / 2 - wheel_radius) }" />
+            <axis xyz="0 1 0" />
+        </joint>
+        <gazebo reference="${name}_wheel">
+            <material>Gazebo/Red</material>
+        </gazebo>
     </xacro:macro>
     <xacro:add_back_wheels name="left_back" flag="1" />
